File: Kicad_project/motocounter/motocounter.kicad_pcb (KiCad board)
At the start: 2 copper layers, 51.6 x 30.9 mm, 53 parts, among them J1 Conn_01x02_Socket, Q1 AO3400A, Q2 AO3401A, U1 L7805, U2 AT24CS02-STUM, U3 AMS1117-3.3, U4 STM32G030F6Px

Commit message: update 12/11
Parts:
- R7: value 1k -> 10k
Changed lines of the file:
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@@
 			)
 		)
-		(property "Value" "1k"
+		(property "Value" "10k"
 			(at 0 1.65 0)
 			(layer "F.Fab")
