File: Kicad_project/motocounter/motocounter.kicad_sch (KiCad schematic)
At the start: 53 parts, among them J1 Conn_01x02_Socket, Q1 AO3400A, Q2 AO3401A, U1 L7805, U2 AT24CS02-STUM, U3 AMS1117-3.3, U4 STM32G030F6Px

Commit message: update 30/11
Parts:
- renumbered S1 to Joystick
Changed lines of the file:
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@@
 	)
 	(junction
+		(at 179.07 72.39)
+		(diameter 0)
+		(color 0 0 0 0)
+	)
+	(junction
 		(at 95.25 71.12)
 		(diameter 0)
@@
 	)
 	(junction
-		(at 181.61 72.39)
-		(diameter 0)
-		(color 0 0 0 0)
-	)
-	(junction
 		(at 114.3 41.91)
 		(diameter 0)
@@
 	(wire
 		(pts
-			(xy 181.61 64.77) (xy 181.61 72.39)
+			(xy 179.07 64.77) (xy 179.07 72.39)
 		)
 		(stroke
@@
 	(wire
 		(pts
-			(xy 180.34 64.77) (xy 181.61 64.77)
+			(xy 176.53 64.77) (xy 179.07 64.77)
 		)
 		(stroke
@@
 	(wire
 		(pts
-			(xy 175.26 72.39) (xy 181.61 72.39)
-		)
-		(stroke
-			(width 0)
-			(type default)
-		)
-	)
-	(wire
-		(pts
 			(xy 67.31 44.45) (xy 67.31 46.99)
 		)
@@
 	(wire
 		(pts
+			(xy 179.07 72.39) (xy 186.69 72.39)
+		)
+		(stroke
+			(width 0)
+			(type default)
+		)
+	)
+	(wire
+		(pts
 			(xy 255.27 29.21) (xy 255.27 31.75)
 		)
@@
 	(wire
 		(pts
-			(xy 181.61 72.39) (xy 186.69 72.39)
-		)
-		(stroke
-			(width 0)
-			(type default)
-		)
-	)
-	(wire
-		(pts
 			(xy 130.81 77.47) (xy 139.7 77.47)
 		)
@@
 	(wire
 		(pts
+			(xy 175.26 72.39) (xy 179.07 72.39)
+		)
+		(stroke
+			(width 0)
+			(type default)
+		)
+	)
+	(wire
+		(pts
 			(xy 66.04 82.55) (xy 77.47 82.55)
 		)
@@
 	(global_label "LED_display"
 		(shape output)
-		(at 180.34 64.77 180)
+		(at 176.53 64.77 180)
 		(fields_autoplaced yes)
 		(effects
@@
 		)
 		(property "Intersheetrefs" "${INTERSHEET_REFS}"
-			(at 166.2274 64.77 0)
+			(at 162.4174 64.77 0)
 			(effects
 				(font
@@
 		(on_board yes)
 		(dnp no)
-		(property "Reference" "S1"
-			(at 113.03 122.936 0)
+		(property "Reference" "Joystick"
+			(at 113.538 127.254 0)
 			(effects
 				(font
@@
 			(project ""
 				(path "/9c61d7ab-836b-4446-b824-a0877c88d6c4"
-					(reference "S1")
+					(reference "Joystick")
 					(unit 1)
 				)

Commit message: update 12/11
Parts:
- R7: value 1k -> 10k
Changed lines of the file:
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@@
 			)
 		)
-		(property "Value" "1k"
+		(property "Value" "10k"
 			(at 147.574 74.422 0)
 			(effects
